Commit message: Attach lidar_link to camera_link (wrong parent)

File: src/course_description/urdf/vehicle.urdf.xacro (robot description, xacro)
@@ -120,5 +120,5 @@
   </link>
   <joint name="lidar_joint" type="fixed">
-    <parent link="base_link"/>
+    <parent link="camera_link"/>
     <child link="lidar_link"/>
     <origin xyz="${sensor_x} 0 ${sensor_z}"/>

Commit message: Attach lidar_link back to base_link

File: src/course_description/urdf/vehicle.urdf.xacro (robot description, xacro)
@@ -120,5 +120,5 @@
   </link>
   <joint name="lidar_joint" type="fixed">
-    <parent link="camera_link"/>
+    <parent link="base_link"/>
     <child link="lidar_link"/>
     <origin xyz="${sensor_x} 0 ${sensor_z}"/>
